Commit message: update robot model

File: examples/robots/sawyer_roller.urdf (robot description, URDF)
Before this commit: robot sawyer, 26 links, 25 joints
Links:
- link finger_left_tip: geometry collision mesh filename=../wsg50/digit.STL; visual cylinder length=0.05 radius=0.02
- link finger_right: geometry collision mesh filename=../wsg50/DIGIT-WSG-50-V1.STL scale=0.001 0.001 0.001; visual mesh filename=../wsg50/DIGIT-WSG-50-V1.STL scale=0.001 0.001 0.001
- link finger_right_tip: geometry collision mesh filename=../wsg50/digit.STL; visual cylinder length=0.05 radius=0.02
- link gripper_base_link: geometry collision mesh filename=../wsg50/WSG50_110.stl scale=1 1 1; visual mesh filename=../wsg50/WSG50_110.stl scale=1 1 1
- link gripper_right: geometry collision mesh filename=../wsg50/GUIDE_WSG50_110.stl scale=0.001 0.001 0.001; visual mesh filename=../wsg50/GUIDE_WSG50_110.stl scale=0.001 0.001 0.001
- link head: geometry collision sphere radius=0.18; visual mesh filename=../sawyer_robot/sawyer_description/meshes/sawyer_pv/head.STL
- link pedestal: geometry collision cylinder length=0.62 radius=0.18; visual mesh filename=../sawyer_robot/sawyer_description/meshes/sawyer_pv/pedesta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
- link right_arm_base_link: geometry collision cylinder length=0.24 radius=0.08; visual mesh filename=../sawyer_robot/sawyer_description/meshes/sawyer_pv/base.DAE
- link right_l0: geometry collision sphere radius=0.07; visual mesh filename=../sawyer_robot/sawyer_description/meshes/sawyer_mp3/l0.DAE
- link right_l1: geometry collision sphere radius=0.07; visual mesh filename=../sawyer_robot/sawyer_description/meshes/sawyer_mp3/l1.DAE
- link right_l2: geometry collision cylinder length=0.35 radius=0.06; visual mesh filename=../sawyer_robot/sawyer_description/meshes/sawyer_pv/l2.DAE
- link right_l3: geometry collision sphere radius=0.06; visual mesh filename=../sawyer_robot/sawyer_description/meshes/sawyer_pv/l3.DAE
- link right_l4: geometry collision cylinder length=0.36 radius=0.045; visual mesh filename=../sawyer_robot/sawyer_description/meshes/sawyer_pv/l4.DAE
- link right_l5: geometry collision sphere radius=0.06; visual mesh filename=../sawyer_robot/sawyer_description/meshes/sawyer_pv/l5.STL
- link right_l6: geometry collision cylinder length=0.05 radius=0.065; visual mesh filename=../sawyer_robot/sawyer_description/meshes/sawyer_mp1/l6.STL

Commit message: update robot model

File: examples/robots/sawyer_roller.urdf (robot description, URDF)
Before this commit: robot sawyer, 26 links, 25 joints
Joints:
- joint base_joint_gripper_left: limit lower=-0.15 upper=-0.0027 effort=1.0 velocity=1.0 -> lower=-0.15 upper=-0.0027 effort=100.0 velocity=100.0
- joint base_joint_gripper_right: limit lower=0.0027 upper=0.15 effort=1.0 velocity=1.0 -> lower=0.0027 upper=0.15 effort=100.0 velocity=100.0

Commit message: add new gripper

File: examples/robots/sawyer_roller.urdf (robot description, URDF)
Before this commit: robot sawyer, 26 links, 25 joints
Links:
- removed link finger_left
- removed link finger_left_tip
- removed link finger_right
- removed link finger_right_tip
- removed link gripper_base_link
- removed link gripper_left
- removed link gripper_right
- added link baselink, mass 0.1; collision cylinder length=0.05325 radius=0.0375; visual cylinder length=0.05325 radius=0.0375
- added link baselink_rx, mass 0.1
- added link baselink_ry, mass 0.1
- added link baselink_rz, mass 0.1
- added link baselink_x, mass 0
- added link baselink_y, mass 0.1
- added link baselink_z, mass 0.1
- added link link1_left, mass 0.005
- added link link1_right, mass 0.005
- added link link2_left, mass 0.005
- added link link2_right, mass 0.005
- added link link3_left, mass 0.01
- added link link3_right, mass 0.01
- added link link4_left, mass 0.005; collision mesh filename=gelsight_cad.obj scale=1 1 1; visual box size=0.01 0.03 0.01
- added link link4_right, mass 0.005; collision mesh filename=gelsight_cad.obj scale=1 1 1; visual box size=0.01 0.03 0.01
Joints:
- removed joint arm_gripper_joint
- removed joint base_joint_gripper_left
- removed joint base_joint_gripper_right
- removed joint guide_joint_finger_left
- removed joint guide_joint_finger_right
- removed joint joint_finger_tip_left
- removed joint joint_finger_tip_right
- added joint baselink_rx: type revolute, parent baselink_rx, child baselink_ry, origin xyz=0 0 0 rpy=0 0 0, axis 1 0 0, limit lower=-10 upper=10 effort=1.0 velocity=10000
- added joint baselink_ry: type revolute, parent baselink_ry, child baselink_rz, origin xyz=0 0 0 rpy=0 0 0, axis 0 1 0, limit lower=-10 upper=10 effort=1.0 velocity=10000
- added joint baselink_rz: type revolute, parent baselink_rz, child baselink, origin xyz=0 0 0 rpy=0 0 0, axis 0 0 1, limit lower=-10 upper=10 effort=1.0 velocity=10000
- added joint baselink_x: type fixed, parent right_hand, child baselink_x, origin xyz=0.0 0.0 0.0 rpy=0.0 0.0 1.5708
- added joint baselink_y: type prismatic, parent baselink_y, child baselink_z, origin xyz=0 0 0 rpy=0 0 0, axis 0 1 0, limit lower=-1 upper=1 effort=1.0 velocity=10000
- added joint baselink_z: type prismatic, parent baselink_z, child baselink_rx, origin xyz=0 0 0 rpy=0 0 0, axis 0 0 1, limit lower=-1 upper=1 effort=1.0 velocity=10000
- added joint joint1_left: type prismatic, parent baselink, child link1_left, origin xyz=0.0 -0.02975 0.05325 rpy=0 0 0, axis 0 0 1, limit lower=-0.06 upper=0 effort=0.1 velocity=10000
- added joint joint1_right: type prismatic, parent baselink, child link1_right, origin xyz=0.0 0.02975 0.05325 rpy=0 0 0, axis 0 0 1, limit lower=-0.06 upper=0 effort=0.1 velocity=10000
- added joint joint2_left: type prismatic, parent link1_left, child link2_left, origin xyz=0.0 0 0.0 rpy=0 0 0, axis 0 1 0, limit lower=-0.06 upper=0 effort=0.1 velocity=10000
- added joint joint2_right: type prismatic, parent link1_right, child link2_right, origin xyz=0.0 0 0.0 rpy=0 0 0, axis 0 1 0, limit lower=0 upper=0.06 effort=0.1 velocity=10000
- added joint joint3_left: type revolute, parent link2_left, child link3_left, origin xyz=0.0 -0.0262 0.08705 rpy=0 0 0, axis 0 1 0, limit lower=-10000 upper=10000 effort=1.0 velocity=10000
- added joint joint3_right: type revolute, parent link2_right, child link3_right, origin xyz=0.0 0.0262 0.08705 rpy=0 0 0, axis 0 1 0, limit lower=-10000 upper=10000 effort=1.0 velocity=10000
- added joint joint4_left: type revolute, parent link3_left, child link4_left, origin xyz=0.0 0.0368 0.0 rpy=0 0 0, axis 0 0 1, limit lower=-10000 upper=10000 effort=1000.0 velocity=10000
- added joint joint4_right: type revolute, parent link3_right, child link4_right, origin xyz=0.0 -0.0368 0.0 rpy=0 0 0, axis 0 0 1, limit lower=-10000 upper=10000 effort=1000.0 velocity=10000

Commit message: add roller env

File: examples/robots/sawyer_roller.urdf (robot description, URDF)
Before this commit: robot sawyer, 28 links, 27 joints
Joints:
- joint roller_baselink_x: origin xyz=0.0 0.0 0.0 rpy=0.0 0.0 1.5708 -> xyz=0.0 0.0 0.0 rpy=0.0 0 0

Commit message: move prismaticly

File: examples/robots/sawyer_roller.urdf (robot description, URDF)
Before this commit: robot sawyer, 28 links, 27 joints
Joints:
- joint joint1_left: axis 1 0 0 -> 0 1 0; limit lower=-10000 upper=10000 effort=1.0 velocity=10000 -> lower=-0.05 upper=0.0 effort=10.0 velocity=10000; type revolute -> prismatic
- joint joint1_right: axis 1 0 0 -> 0 1 0; limit lower=-10000 upper=10000 effort=1.0 velocity=10000 -> lower=0.0 upper=0.05 effort=10.0 velocity=10000; type revolute -> prismatic
- joint joint2_left: type revolute -> fixed
- joint joint2_right: type revolute -> fixed
